Commit message: Updated project name and rviz views

File: dataset_tools/ros2/cu_multi_ros2_ws/src/cu_multi_ros2/urdf/multi_robot.urdf (robot description, URDF)
Before this commit: robot hunter_robot, 19 links, 18 joints
Links:
- link robotf_camera_link: geometry collision cylinder length=0.0742 radius=0.0435; visual mesh filename=package://cu_multi_ros/urdf/meshes/dae/d435.dae scale=1.0 1.0 1.0
- link robotf_chassis: geometry collision mesh filename=package://cu_multi_ros/urdf/meshes/dae/hunter_base.dae scale=1.0 1.0 1.0; visual mesh filename=package://cu_multi_ros/urdf/meshes/dae/hunter_base.dae scale=1.0 1.0 1.0
- link robotf_left_front_wheel: geometry collision cylinder length=0.08912 radius=0.1375; visual mesh filename=package://cu_multi_ros/urdf/meshes/dae/hunter_wheel.dae scale=-0.001 0.001 0.001
- link robotf_left_rear_wheel: geometry collision cylinder length=0.08912 radius=0.1375; visual mesh filename=package://cu_multi_ros/urdf/meshes/dae/hunter_wheel.dae scale=-0.001 0.001 0.001
- link robotf_os_sensor: geometry collision cylinder length=0.0742 radius=0.0435; visual mesh filename=package://cu_multi_ros/urdf/meshes/dae/os_sensor.dae scale=-0.001 0.001 0.001
- link robotf_right_front_wheel: geometry collision cylinder length=0.08912 radius=0.1375; visual mesh filename=package://cu_multi_ros/urdf/meshes/dae/hunter_wheel.dae scale=-0.001 0.001 0.001
- link robotf_right_rear_wheel: geometry collision cylinder length=0.08912 radius=0.1375; visual mesh filename=package://cu_multi_ros/urdf/meshes/dae/hunter_wheel.dae scale=-0.001 0.001 0.001

File: dataset_tools/ros2/cu_multi_ros2_ws/src/cu_multi_ros2/urdf/multi_robot.urdf.xacro (robot description, xacro)
@@ -120,5 +120,5 @@
         <origin xyz="0 ${lr_reflect*(axle_length-(tire_width/2-hex_hub_depth))} 0" rpy="${degrees_90 + lr_reflect*degrees_90} 0 0"/>
         <geometry>
-		      <mesh filename="package://lidar2osm_ros/urdf/meshes/dae/hunter_wheel.dae"  scale="-0.001 0.001 0.001"/>
+		      <mesh filename="package://cu_multi_ros/urdf/meshes/dae/hunter_wheel.dae"  scale="-0.001 0.001 0.001"/>
         </geometry>
         <material name="tire_mat"/>
@@ -127,5 +127,5 @@
         <origin xyz="0 ${lr_reflect*(axle_length-(tire_width/2-hex_hub_depth))} 0"/>
         <geometry>
-          <!-- <mesh filename="package://lidar2osm_ros/urdf/meshes/back-wheel-no-axel_c.stl"  scale="-0.001 0.001 0.001"/> -->
+          <!-- <mesh filename="package://cu_multi_ros/urdf/meshes/back-wheel-no-axel_c.stl"  scale="-0.001 0.001 0.001"/> -->
           <cylinder radius="${tire_dia/2}" length="${tire_width}"/>
         </geometry>
@@ -173,6 +173,6 @@
       <origin xyz="0 0 ${-chassis_height / 2}" rpy="0 0 ${degrees_90}"/>
       <geometry>
-        <!-- <mesh filename="package://lidar2osm_ros/urdf/meshes/dae/hunter_base.dae"  scale="0.0055 0.0055 0.0055"/> -->
-        <mesh filename="package://lidar2osm_ros/urdf/meshes/dae/hunter_base.dae"  scale="1.0 1.0 1.0"/>
+        <!-- <mesh filename="package://cu_multi_ros/urdf/meshes/dae/hunter_base.dae"  scale="0.0055 0.0055 0.0055"/> -->
+        <mesh filename="package://cu_multi_ros/urdf/meshes/dae/hunter_base.dae"  scale="1.0 1.0 1.0"/>
       </geometry>
       <material name="chassis_mat"/>
@@ -181,5 +181,5 @@
       <origin xyz="0 0 ${-chassis_height / 2}"/>
       <geometry>
-        <mesh filename="package://lidar2osm_ros/urdf/meshes/dae/hunter_base.dae"  scale="1.0 1.0 1.0"/>
+        <mesh filename="package://cu_multi_ros/urdf/meshes/dae/hunter_base.dae"  scale="1.0 1.0 1.0"/>
       </geometry>
     </collision>
@@ -215,5 +215,5 @@
         <origin xyz="-0.045 0.04 ${-ouster_height/2}" rpy="${degrees_90} 0 ${degrees_90}"/>
         <geometry>
-          <mesh filename="package://lidar2osm_ros/urdf/meshes/dae/os_sensor.dae"  scale="-0.001 0.001 0.001"/>
+          <mesh filename="package://cu_multi_ros/urdf/meshes/dae/os_sensor.dae"  scale="-0.001 0.001 0.001"/>
         </geometry>
         <material name="chassis_mat"/>
@@ -266,5 +266,5 @@
         <origin xyz="0.00 0.00 0.00" rpy="${degrees_90} 0 ${degrees_90}"/>
         <geometry>
-          <mesh filename="package://lidar2osm_ros/urdf/meshes/dae/d435.dae"  scale="1.0 1.0 1.0"/>
+          <mesh filename="package://cu_multi_ros/urdf/meshes/dae/d435.dae"  scale="1.0 1.0 1.0"/>
         </geometry>
       </visual>

File: dataset_tools/ros2/cu_multi_ros2_ws/src/cu_multi_ros2/urdf/multi_robot_IMU.urdf.xacro (robot description, xacro)
@@ -111,5 +111,5 @@
         <origin xyz="0 ${lr_reflect*(axle_length-(tire_width/2-hex_hub_depth))} 0" rpy="${degrees_90 + lr_reflect*degrees_90} 0 0"/>
         <geometry>
-		      <mesh filename="package://lidar2osm_ros/urdf/meshes/dae/hunter_wheel.dae"  scale="-0.001 0.001 0.001"/>
+		      <mesh filename="package://cu_multi_ros/urdf/meshes/dae/hunter_wheel.dae"  scale="-0.001 0.001 0.001"/>
         </geometry>
         <material name="tire_mat"/>
@@ -170,5 +170,5 @@
         <origin xyz="-0.045 0.04 ${-ouster_height/2}" rpy="${degrees_90} 0 ${degrees_90}"/>
         <geometry>
-          <mesh filename="package://lidar2osm_ros/urdf/meshes/dae/os_sensor.dae"  scale="-0.001 0.001 0.001"/>
+          <mesh filename="package://cu_multi_ros/urdf/meshes/dae/os_sensor.dae"  scale="-0.001 0.001 0.001"/>
         </geometry>
         <material name="chassis_mat"/>

File: dataset_tools/ros2/cu_multi_ros2_ws/src/cu_multi_ros2/urdf/single_robot.urdf.xacro (robot description, xacro)
@@ -120,5 +120,5 @@
         <origin xyz="0 ${lr_reflect*(axle_length-(tire_width/2-hex_hub_depth))} 0" rpy="${degrees_90 + lr_reflect*degrees_90} 0 0"/>
         <geometry>
-		      <mesh filename="package://lidar2osm_ros/urdf/meshes/dae/hunter_wheel.dae"  scale="-0.001 0.001 0.001"/>
+		      <mesh filename="package://cu_multi_ros/urdf/meshes/dae/hunter_wheel.dae"  scale="-0.001 0.001 0.001"/>
         </geometry>
         <material name="tire_mat"/>
@@ -127,5 +127,5 @@
         <origin xyz="0 ${lr_reflect*(axle_length-(tire_width/2-hex_hub_depth))} 0"/>
         <geometry>
-          <!-- <mesh filename="package://lidar2osm_ros/urdf/meshes/back-wheel-no-axel_c.stl"  scale="-0.001 0.001 0.001"/> -->
+          <!-- <mesh filename="package://cu_multi_ros/urdf/meshes/back-wheel-no-axel_c.stl"  scale="-0.001 0.001 0.001"/> -->
           <cylinder radius="${tire_dia/2}" length="${tire_width}"/>
         </geometry>
@@ -173,6 +173,6 @@
       <origin xyz="0 0 ${-chassis_height / 2}" rpy="0 0 ${degrees_90}"/>
       <geometry>
-        <!-- <mesh filename="package://lidar2osm_ros/urdf/meshes/dae/hunter_base.dae"  scale="0.0055 0.0055 0.0055"/> -->
-        <mesh filename="package://lidar2osm_ros/urdf/meshes/dae/hunter_base.dae"  scale="1.0 1.0 1.0"/>
+        <!-- <mesh filename="package://cu_multi_ros/urdf/meshes/dae/hunter_base.dae"  scale="0.0055 0.0055 0.0055"/> -->
+        <mesh filename="package://cu_multi_ros/urdf/meshes/dae/hunter_base.dae"  scale="1.0 1.0 1.0"/>
       </geometry>
       <material name="chassis_mat"/>
@@ -181,5 +181,5 @@
       <origin xyz="0 0 ${-chassis_height / 2}"/>
       <geometry>
-        <mesh filename="package://lidar2osm_ros/urdf/meshes/dae/hunter_base.dae"  scale="1.0 1.0 1.0"/>
+        <mesh filename="package://cu_multi_ros/urdf/meshes/dae/hunter_base.dae"  scale="1.0 1.0 1.0"/>
       </geometry>
     </collision>
@@ -215,5 +215,5 @@
         <origin xyz="-0.045 0.04 ${-ouster_height/2}" rpy="${degrees_90} 0 ${degrees_90}"/>
         <geometry>
-          <mesh filename="package://lidar2osm_ros/urdf/meshes/dae/os_sensor.dae"  scale="-0.001 0.001 0.001"/>
+          <mesh filename="package://cu_multi_ros/urdf/meshes/dae/os_sensor.dae"  scale="-0.001 0.001 0.001"/>
         </geometry>
         <material name="chassis_mat"/>
@@ -266,5 +266,5 @@
         <origin xyz="0.00 0.00 0.00" rpy="${degrees_90} 0 ${degrees_90}"/>
         <geometry>
-          <mesh filename="package://lidar2osm_ros/urdf/meshes/dae/d435.dae"  scale="1.0 1.0 1.0"/>
+          <mesh filename="package://cu_multi_ros/urdf/meshes/dae/d435.dae"  scale="1.0 1.0 1.0"/>
         </geometry>
       </visual>
